File: schematics/tian_light_rgb_revc.sch (EAGLE design)
At the start: 7 parts

Commit message: -a
Parts:
- removed C1: (no value), rcl:CPOL-EU153CLV-0605
- added C2: 220uF, rcl:CPOL-EUF
- added F1: (no value), fuse:SH22,5
Connections:
- new net N$1: F1.1, X1-1.KL
- net 12V: now also C2.+, F1.2; no longer C1.+, X1-1.KL
- net GND: now also C2.-; no longer C1.-
Other:
- note added: "FUSE (OPTIONAL)"
- note added: "SMD"
Changed lines of the file:
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@@
 <part name="U$3" library="tian" deviceset="BUCK_LED_DRIVER" device=""/>
 <part name="U$5" library="strukt" deviceset="1PORT_ETHERNET" device=""/>
-<part name="C1" library="rcl" deviceset="CPOL-EU" device="153CLV-0605"/>
 <part name="X1" library="con-wago-508" deviceset="W237-02P" device=""/>
-<part name="P+1" library="SparkFun" deviceset="VCC" device=""/>
 <part name="GND2" library="SparkFun" deviceset="GND" device=""/>
+<part name="F1" library="fuse" deviceset="SH22,5" device=""/>
+<part name="P+2" library="SparkFun" deviceset="VCC" device=""/>
+<part name="C2" library="rcl" deviceset="CPOL-EU" device="F" value="220uF"/>
 </parts>
 <sheets>
@@
 <text x="45.72" y="91.44" size="2.54" layer="91">LED DRIVER</text>
 <text x="180.34" y="99.06" size="1.778" layer="91">achtung: steckerbelegung anders als bei rev.B!!!</text>
+<text x="185.42" y="134.62" size="1.778" layer="91" rot="R90">FUSE (OPTIONAL)</text>
+<text x="124.46" y="144.78" size="1.778" layer="91" rot="R90">SMD</text>
 </plain>
 <instances>
 <instance part="P+4" gate="1" x="127" y="149.86"/>
-<instance part="GND7" gate="1" x="127" y="124.46"/>
+<instance part="GND7" gate="1" x="127" y="129.54"/>
 <instance part="FRAME1" gate="G$1" x="0" y="0"/>
 <instance part="U$1" gate="G$1" x="40.64" y="132.08"/>
@@
 <instance part="U$3" gate="G$1" x="40.64" y="66.04"/>
 <instance part="U$5" gate="1PORTRJ45" x="152.4" y="71.12"/>
-<instance part="C1" gate="G$1" x="127" y="142.24"/>
 <instance part="X1" gate="-1" x="170.18" y="139.7"/>
 <instance part="X1" gate="-2" x="170.18" y="134.62"/>
-<instance part="P+1" gate="1" x="182.88" y="154.94"/>
 <instance part="GND2" gate="1" x="180.34" y="124.46"/>
+<instance part="F1" gate="1" x="180.34" y="147.32" rot="R90"/>
+<instance part="P+2" gate="1" x="180.34" y="157.48"/>
+<instance part="C2" gate="G$1" x="127" y="142.24"/>
 </instances>
 <busses>
@@
 <segment>
 <pinref part="GND7" gate="1" pin="GND"/>
-<pinref part="C1" gate="G$1" pin="-"/>
-<wire x1="127" y1="132.08" x2="127" y2="127" width="0.1524" layer="91"/>
-<wire x1="127" y1="132.08" x2="127" y2="134.62" width="0.1524" layer="91"/>
-<wire x1="127" y1="134.62" x2="127" y2="137.16" width="0.1524" layer="91"/>
+<wire x1="127" y1="132.08" x2="127" y2="137.16" width="0.1524" layer="91"/>
+<pinref part="C2" gate="G$1" pin="-"/>
 </segment>
 <segment>
@@
 <segment>
 <pinref part="P+4" gate="1" pin="VCC"/>
-<pinref part="C1" gate="G$1" pin="+"/>
 <wire x1="127" y1="149.86" x2="127" y2="144.78" width="0.1524" layer="91"/>
+<pinref part="C2" gate="G$1" pin="+"/>
 </segment>
 <segment>
@@
 </segment>
 <segment>
-<pinref part="X1" gate="-1" pin="KL"/>
-<wire x1="175.26" y1="139.7" x2="180.34" y2="139.7" width="0.1524" layer="91"/>
-<wire x1="180.34" y1="139.7" x2="180.34" y2="152.4" width="0.1524" layer="91"/>
-<pinref part="P+1" gate="1" pin="VCC"/>
-<wire x1="180.34" y1="152.4" x2="182.88" y2="154.94" width="0.1524" layer="91"/>
+<pinref part="P+2" gate="1" pin="VCC"/>
+<pinref part="F1" gate="1" pin="2"/>
+<wire x1="180.34" y1="157.48" x2="180.34" y2="152.4" width="0.1524" layer="91"/>
 </segment>
 </net>
@@
 <pinref part="X3" gate="-2" pin="KL"/>
 <wire x1="223.52" y1="66.04" x2="182.88" y2="66.04" width="0.1524" layer="91"/>
-<label x="185.42" y="66.04" size="1.778" layer="95"/>
+<label x="182.88" y="66.04" size="1.778" layer="95"/>
 </segment>
 </net>
@@
 <pinref part="X3" gate="-4" pin="KL"/>
 <wire x1="223.52" y1="76.2" x2="182.88" y2="76.2" width="0.1524" layer="91"/>
-<label x="185.42" y="76.2" size="1.778" layer="95"/>
+<label x="182.88" y="76.2" size="1.778" layer="95"/>
 </segment>
 </net>
@@
 <pinref part="X3" gate="-5" pin="KL"/>
 <wire x1="223.52" y1="81.28" x2="182.88" y2="81.28" width="0.1524" layer="91"/>
-<label x="185.42" y="81.28" size="1.778" layer="95"/>
+<label x="182.88" y="81.28" size="1.778" layer="95"/>
 </segment>
 </net>
@@
 <pinref part="X3" gate="-1" pin="KL"/>
 <wire x1="223.52" y1="60.96" x2="182.88" y2="60.96" width="0.1524" layer="91"/>
-<label x="185.42" y="60.96" size="1.778" layer="95"/>
+<label x="182.88" y="60.96" size="1.778" layer="95"/>
 </segment>
 </net>
@@
 <pinref part="X3" gate="-3" pin="KL"/>
 <wire x1="223.52" y1="71.12" x2="182.88" y2="71.12" width="0.1524" layer="91"/>
-<label x="185.42" y="71.12" size="1.778" layer="95"/>
+<label x="182.88" y="71.12" size="1.778" layer="95"/>
+</segment>
+</net>
+<net name="N$1" class="0">
+<segment>
+<pinref part="X1" gate="-1" pin="KL"/>
+<wire x1="175.26" y1="139.7" x2="180.34" y2="139.7" width="0.1524" layer="91"/>
+<pinref part="F1" gate="1" pin="1"/>
+<wire x1="180.34" y1="142.24" x2="180.34" y2="139.7" width="0.1524" layer="91"/>
 </segment>
 </net>
@@
 </sheet>
 </sheets>
+<errors>
+</errors>
 </schematic>
 </drawing>
